File: Mainboard/DS01A-3.kicad_pcb (KiCad board)
At the start: 2 copper layers, 152 x 162 mm, 80 parts, among them CON1 Floppy Drive Connector, J1 Barrel_Jack, U5X1 Alternate U5, U6S1 Alternate U6, U9 27C256 PLCC-32

Commit message: Add files via upload
Parts:
- moved CN2 0.45 mm to (195.2, 138.2)
Routing:
- net /~{WRAM}: track 148.0 -> 150.6 mm
- net /D0.Sys: track 473.2 -> 475.7 mm
- net /L.Audio: track 20.1 -> 18.2 mm
- net /EXPAND: track 133.4 -> 135.1 mm
- net /~{PAWR}: track 127.2 -> 128.8 mm
- net /D1.Sys: track 453.2 -> 454.8 mm
- net /PA6: track 128.6 -> 130.1 mm
- net /D2.Sys: track 470.3 -> 471.6 mm
- net /D5.Sys: track 439.8 -> 441.0 mm
- net /D4.Sys: track 476.8 -> 478.0 mm
- net /PA7: track 148.1 -> 149.1 mm
- net /D3.Sys: track 435.1 -> 436.0 mm
- net /~{PARD}: track 124.6 -> 125.5 mm
- net /REFRESH: track 134.1 -> 134.9 mm
- net /~{CS}.U5: track 120.4 -> 120.9 mm
Other:
- outline, holes or cut-outs redrawn
