File: Memory Addon Board/Memory Board.kicad_pcb (KiCad board)
At the start: 2 copper layers, 59 x 30.5 mm, 8 parts

Commit message: Add files via upload
Parts:
- C1, C2: value 100 nF -> 100 pF
Connections:
- C1 pad 2: /VREG.5V -> /~{CAS}.RAM1-3
- C2 pad 2: /VREG.5V -> /~{CAS}.RAM2-4
Routing:
- net /D6.Sys: track 94.4 -> 68.1 mm
- net /~{CAS}.RAM1-3: track 55.6 -> 78.2 mm, vias 1 -> 2
- net /A8.RAM: track 72.6 -> 94.5 mm, vias 2 -> 1
- net /A9.RAM: track 90.3 -> 70.8 mm, vias 3 -> 2
- net /A3.RAM: track 99.6 -> 80.2 mm, vias 4 -> 1
- net /A1.RAM: track 85.0 -> 101.6 mm, vias 4 -> 1
- net /VREG.5V: track 142.2 -> 127.6 mm, vias 6 -> 3
- net /A0.RAM: track 82.0 -> 67.7 mm, vias 4 -> 2
- net /D2.Sys: track 97.6 -> 83.6 mm, vias 4 -> 1
- net /~{OE}.RAM3: track 53.7 -> 40.2 mm
- net /A4.RAM: track 82.9 -> 95.7 mm, vias 1 -> 3
- net /A2.RAM: track 88.9 -> 76.9 mm, vias 3 -> 1
- net /D0.Sys: track 89.1 -> 77.6 mm, vias 3 -> 1
- net /~{OE}.RAM2: track 43.5 -> 51.1 mm
- net /A5.RAM: track 75.1 -> 82.6 mm, vias 2 -> 5
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