File: Memory Addon Board/Memory Board.kicad_sch (KiCad schematic)
At the start: 8 parts

Commit message: Add files via upload
Parts:
- C1, C2: value 100 nF -> 100 pF
Connections:
- net VREG.5V: no longer C1.2, C2.2
- net ~{CAS}.RAM1-3: now also C1.2
- net ~{CAS}.RAM2-4: now also C2.2
Other:
- moved on the sheet: C1, C2
Changed lines of the file:
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@@
+	)
+	(label "~{CAS}.RAM2-4"
+		(at 157.48 85.09 90)
+		(fields_autoplaced yes)
+		(effects
+			(font
+				(size 1.27 1.27)
+			)
+			(justify left bottom)
+		)
 	)
 	(label "~{CAS}.RAM2-4"
@@
 		)
 	)
+	(label "~{CAS}.RAM1-3"
+		(at 133.35 85.09 90)
+		(fields_autoplaced yes)
+		(effects
+			(font
+				(size 1.27 1.27)
+			)
+			(justify left bottom)
+		)
+	)
 	(label "VREG.5V"
 		(at 67.31 138.43 180)
@@
 	)
 	(label "GND"
-		(at 144.78 88.9 270)
+		(at 133.35 90.17 270)
 		(fields_autoplaced yes)
 		(effects
@@
 		)
 	)
-	(label "VREG.5V"
-		(at 168.91 83.82 90)
-		(fields_autoplaced yes)
-		(effects
-			(font
-				(size 1.27 1.27)
-			)
-			(justify left bottom)
-		)
-	)
 	(label "D6.Sys"
 		(at 165.1 115.57 180)
@@
 	)
 	(label "GND"
-		(at 168.91 88.9 270)
+		(at 157.48 90.17 270)
 		(fields_autoplaced yes)
 		(effects
@@
 			)
 			(justify right bottom)
-		)
-	)
-	(label "VREG.5V"
-		(at 144.78 83.82 90)
-		(fields_autoplaced yes)
-		(effects
-			(font
-				(size 1.27 1.27)
-			)
-			(justify left bottom)
 		)
 	)
@@
 	(symbol
 		(lib_id "Device:C_Small")
-		(at 144.78 86.36 0)
+		(at 133.35 87.63 0)
 		(mirror x)
 		(unit 1)
@@
 		(fields_autoplaced yes)
 		(property "Reference" "C1"
-			(at 142.24 85.0835 0)
+			(at 130.81 86.3535 0)
 			(effects
 				(font
@@
 			)
 		)
-		(property "Value" "100 nF"
-			(at 142.24 87.6235 0)
+		(property "Value" "100 pF"
+			(at 130.81 88.8935 0)
 			(effects
 				(font
@@
 		)
 		(property "Footprint" "SFIII:SMD Passive"
-			(at 144.78 86.36 0)
+			(at 133.35 87.63 0)
 			(effects
 				(font
@@
 		)
 		(property "Datasheet" "~"
-			(at 144.78 86.36 0)
+			(at 133.35 87.63 0)
 			(effects
 				(font
@@
 		)
 		(property "Description" "0.1u"
-			(at 144.78 86.36 0)
+			(at 133.35 87.63 0)
 			(effects
 				(font
@@
 	(symbol
 		(lib_id "Device:C_Small")
-		(at 168.91 86.36 0)
+		(at 157.48 87.63 0)
 		(mirror x)
 		(unit 1)
@@
 		(fields_autoplaced yes)
 		(property "Reference" "C2"
-			(at 166.37 85.0835 0)
+			(at 154.94 86.3535 0)
 			(effects
 				(font
@@
 			)
 		)
-		(property "Value" "100 nF"
-			(at 166.37 87.6235 0)
+		(property "Value" "100 pF"
+			(at 154.94 88.8935 0)
 			(effects
 				(font
@@
 		)
 		(property "Footprint" "SFIII:SMD Passive"
-			(at 168.91 86.36 0)
+			(at 157.48 87.63 0)
 			(effects
 				(font
@@
 		)
 		(property "Datasheet" "~"
-			(at 168.91 86.36 0)
+			(at 157.48 87.63 0)
 			(effects
 				(font
@@
 		)
 		(property "Description" "0.1u"
-			(at 168.91 86.36 0)
-			(effects
-				(font
+			(at 157.48 87.63 0)
+			(effects
+				(font
